Commit message: AI - working GA

File: L6/cm3020_ai/simscreatures/temp0.urdf (robot description, URDF)
Before this commit: robot pepe, 13 links, 12 joints
Links:
- removed link 15
- removed link 19
- removed link 210
- removed link 211
- removed link 212
- removed link 26
- removed link 27
- removed link 28
- link 0: mass 0.1386419682712971 -> 2.508821932468066; geometry collision cylinder length=1.3027125246961713 radius=0.7829529922033459; visual cylinder length=1.3027125246961713 radius=0.7829529922033459
- link 11: mass 0.9487643918334238 -> 0.21497982086557357; geometry collision cylinder length=1.8843324128801913 radius=0.19056588350260817; visual cylinder length=1.8843324128801913 radius=0.19056588350260817
- link 22: mass 1.0117344253041407 -> 0.004846521487007137; geometry collision cylinder length=0.4618823797775875 radius=0.05779289334218429; visual cylinder length=0.4618823797775875 radius=0.05779289334218429
- link 23: mass 1.0117344253041407 -> 0.004846521487007137; geometry collision cylinder length=0.4618823797775875 radius=0.05779289334218429; visual cylinder length=0.4618823797775875 radius=0.05779289334218429
- link 24: mass 1.0117344253041407 -> 0.004846521487007137; geometry collision cylinder length=0.4618823797775875 radius=0.05779289334218429; visual cylinder length=0.4618823797775875 radius=0.05779289334218429
Joints:
- removed joint 15_to_0
- removed joint 19_to_0
- removed joint 210_to_19
- removed joint 211_to_19
- removed joint 212_to_19
- removed joint 26_to_15
- removed joint 27_to_15
- removed joint 28_to_15
- joint 11_to_0: axis 0 1 0 -> 0 0 1; origin xyz=0.5197156954984278 0.6900856637265136 0.7281011155971425 rpy=2.744312139012575 5.325808283454467 0.6888846513822823 -> xyz=0.4215110883640615 0.2188065997501728 0.9398203673718867 rpy=12.14274553194132 6.046821119140343 5.4519879205980954
- joint 22_to_11: axis 0 1 0 -> 1 0 0; origin xyz=0.4014772245747642 0.9633709495588345 0.9799982140258243 rpy=10.64023491395587 4.143551934509013 3.4519210623905625 -> xyz=0.36952773696045593 0.10836644126601783 0.5477438343449981 rpy=11.854298137734773 5.175247813080558 4.195008801091541
- joint 23_to_11: axis 0 1 0 -> 1 0 0; origin xyz=0.4014772245747642 0.9633709495588345 0.9799982140258243 rpy=15.960352370933805 4.143551934509013 3.4519210623905625 -> xyz=0.36952773696045593 0.10836644126601783 0.5477438343449981 rpy=17.78144720660216 5.175247813080558 4.195008801091541
- joint 24_to_11: axis 0 1 0 -> 1 0 0; origin xyz=0.4014772245747642 0.9633709495588345 0.9799982140258243 rpy=21.28046982791174 4.143551934509013 3.4519210623905625 -> xyz=0.36952773696045593 0.10836644126601783 0.5477438343449981 rpy=23.708596275469546 5.175247813080558 4.195008801091541

File: L6/cm3020_ai/simscreatures/test.urdf (robot description, URDF)
Before this commit: robot pepe, 10 links, 9 joints
Links:
- removed link 14
- removed link 17
- removed link 22
- removed link 23
- removed link 25
- removed link 26
- removed link 28
- removed link 29
- added link 12, mass 2.297918675244149; collision cylinder length=1.134041496494729 radius=0.8031153335333476; visual cylinder length=1.134041496494729 radius=0.8031153335333476
- added link 13, mass 2.297918675244149; collision cylinder length=1.134041496494729 radius=0.8031153335333476; visual cylinder length=1.134041496494729 radius=0.8031153335333476
- link 0: mass 0.023657479216776425 -> 0.2103234233305153; geometry collision cylinder length=0.503183918073304 radius=0.36475857333205775; visual cylinder length=0.503183918073304 radius=0.36475857333205775
- link 11: mass 0.014037622475716379 -> 2.297918675244149; geometry collision cylinder length=1.134041496494729 radius=0.8031153335333476; visual cylinder length=1.134041496494729 radius=0.8031153335333476
Joints:
- removed joint 14_to_0
- removed joint 17_to_0
- removed joint 22_to_11
- removed joint 23_to_11
- removed joint 25_to_14
- removed joint 26_to_14
- removed joint 28_to_17
- removed joint 29_to_17
- added joint 12_to_0: type revolute, parent 0, child 12, origin xyz=0.8166271055768323 0.060541167397329065 0.9999 rpy=11.290049196770866 4.831392402738542 2.270539807682347, axis 1 0 0, limit lower=3.1415 upper=-3.1415 effort=1 velocity=1
- added joint 13_to_0: type revolute, parent 0, child 13, origin xyz=0.8166271055768323 0.060541167397329065 0.9999 rpy=15.053398929027821 4.831392402738542 2.270539807682347, axis 1 0 0, limit lower=3.1415 upper=-3.1415 effort=1 velocity=1
- joint 11_to_0: axis 0 0 1 -> 1 0 0; origin xyz=0.5568495220376454 0.26434843091369065 0.7896240210922013 rpy=1.289679924820228 5.787012117342018 3.5123657341751917 -> xyz=0.8166271055768323 0.060541167397329065 0.9999 rpy=7.526699464513911 4.831392402738542 2.270539807682347

Commit message: AI Midterm done

File: L6/cm3020_ai/simscreatures/temp0.urdf (robot description, URDF)
Before this commit: robot pepe, 5 links, 4 joints
Links:
- removed link 22
- removed link 24
- added link 32, mass 1.6312563707260126; collision cylinder length=0.5193488942877491 radius=0.9999; visual cylinder length=0.5193488942877491 radius=0.9999
- link 0: mass 2.508821932468066 -> 0.09535784327793705; geometry collision cylinder length=0.8669926428735232 radius=0.18710938339079877; visual cylinder length=0.8669926428735232 radius=0.18710938339079877
- link 11: mass 0.21497982086557357 -> 2.2594492440210128; geometry collision cylinder length=0.7193488942877491 radius=0.9999; visual cylinder length=0.7193488942877491 radius=0.9999
- link 23: mass 0.004846521487007137 -> 2.573545680668513; geometry collision cylinder length=0.819348894287749 radius=0.9999; visual cylinder length=0.819348894287749 radius=0.9999
Joints:
- removed joint 22_to_11
- removed joint 23_to_11
- removed joint 24_to_11
- added joint 23_to_0: type revolute, parent 0, child 23, origin xyz=0.9999 0.9999 0.4069430828837445 rpy=9.546168221575648 6.282556988648868 6.282556988648868, axis 0 0 1, limit lower=3.1415 upper=-3.1415 effort=1 velocity=1
- added joint 32_to_11: type revolute, parent 11, child 32, origin xyz=0.9999 0.9999 0.3069430828837445 rpy=5.107475086281181 6.282556988648868 6.282556988648868, axis 0 0 1, limit lower=3.1415 upper=-3.1415 effort=1 velocity=1
- joint 11_to_0: origin xyz=0.4215110883640615 0.2188065997501728 0.9398203673718867 rpy=12.14274553194132 6.046821119140343 5.4519879205980954 -> xyz=0.9999 0.9999 0.5069430828837445 rpy=5.107475086281181 6.282556988648868 6.282556988648868

File: L6/cm3020_ai/simscreatures/temp1.urdf (robot description, URDF)
Before this commit: robot pepe, 1 links, 0 joints
Links:
- added link 11, mass 0.02066784348313888; collision cylinder length=0.8669926428735232 radius=0.08710938339079877; visual cylinder length=0.8669926428735232 radius=0.08710938339079877
- link 0: mass 0.040484087548324665 -> 1.6312563707260126; geometry collision cylinder length=0.5193488942877491 radius=0.9999; visual cylinder length=0.5193488942877491 radius=0.9999
Joints:
- added joint 11_to_0: type revolute, parent 0, child 11, origin xyz=0.8458982153510861 0.7495428260868736 0.2733804451619263 rpy=10.750803443343083 1.7154021787407705 0.757835571468532, axis 0 1 0, limit lower=3.1415 upper=-3.1415 effort=1 velocity=1

File: L6/cm3020_ai/simscreatures/temp2.urdf (robot description, URDF)
Before this commit: robot pepe, 3 links, 2 joints
Links:
- removed link 22
- added link 23, mass 2.2594492440210128; collision cylinder length=0.7193488942877491 radius=0.9999; visual cylinder length=0.7193488942877491 radius=0.9999
- added link 32, mass 1.6312563707260126; collision cylinder length=0.5193488942877491 radius=0.9999; visual cylinder length=0.5193488942877491 radius=0.9999
- added link 44, mass 0.38386024474465524; collision cylinder length=0.31429930265885975 radius=0.6235049746617803; visual cylinder length=0.31429930265885975 radius=0.6235049746617803
- link 0: mass 3.248769649119231 -> 0.010091801124406666; geometry collision cylinder length=0.5230673599617152 radius=0.07836652606024419; visual cylinder length=0.5230673599617152 radius=0.07836652606024419
- link 11: mass 4.439031451905032 -> 0.02066784348313888; geometry collision cylinder length=0.8669926428735232 radius=0.08710938339079877; visual cylinder length=0.8669926428735232 radius=0.08710938339079877
Joints:
- removed joint 22_to_11
- added joint 23_to_0: type revolute, parent 0, child 23, origin xyz=0.9999 0.9999 0.20694308288374447 rpy=9.546168221575648 6.282556988648868 6.282556988648868, axis 0 0 1, limit lower=3.1415 upper=-3.1415 effort=1 velocity=1
- added joint 32_to_11: type revolute, parent 11, child 32, origin xyz=0.9999 0.9999 0.3069430828837445 rpy=5.107475086281181 6.282556988648868 6.282556988648868, axis 0 0 1, limit lower=3.1415 upper=-3.1415 effort=1 velocity=1
- added joint 44_to_0: type revolute, parent 0, child 44, origin xyz=0.528868182730234 0.9829652923630362 0.03029427048696387 rpy=8.280162887455393 1.5492331212387762 2.5357965924058323, axis 0 1 0, limit lower=3.1415 upper=-3.1415 effort=1 velocity=1
- joint 11_to_0: axis 1 0 0 -> 0 1 0; origin xyz=0.2535809368132803 0.5229588186878955 0.14097722991465836 rpy=10.712675389893242 1.5974257988825435 2.223050566148718 -> xyz=0.8458982153510861 0.8495428260868736 0.2733804451619263 rpy=12.007440504779 2.343720709458729 0.757835571468532

File: L6/cm3020_ai/simscreatures/temp3.urdf (robot description, URDF)
Before this commit: robot pepe, 3 links, 2 joints
Links:
- removed link 12
- added link 23, mass 0.02066784348313888; collision cylinder length=0.8669926428735232 radius=0.08710938339079877; visual cylinder length=0.8669926428735232 radius=0.08710938339079877
- added link 32, mass 2.2594492440210128; collision cylinder length=0.7193488942877491 radius=0.9999; visual cylinder length=0.7193488942877491 radius=0.9999
- added link 44, mass 0.013485873308373975; collision cylinder length=0.12443131712763478 radius=0.18573756694812382; visual cylinder length=0.12443131712763478 radius=0.18573756694812382
- link 0: mass 0.6943324061292382 -> 2.2594492440210128; geometry collision cylinder length=0.7193488942877491 radius=0.9999; visual cylinder length=0.7193488942877491 radius=0.9999
- link 11: mass 0.6943324061292382 -> 1.9453528073735127; geometry collision cylinder length=0.6193488942877491 radius=0.9999; visual cylinder length=0.6193488942877491 radius=0.9999
Joints:
- removed joint 12_to_0
- added joint 23_to_0: type revolute, parent 0, child 23, origin xyz=0.8458982153510861 0.8495428260868736 0.37338044516192626 rpy=16.126205165014625 1.7154021787407705 0.757835571468532, axis 0 1 0, limit lower=3.1415 upper=-3.1415 effort=1 velocity=1
- added joint 32_to_11: type revolute, parent 11, child 32, origin xyz=0.9999 0.9999 0.5069430828837445 rpy=5.107475086281181 6.282556988648868 6.282556988648868, axis 0 0 1, limit lower=3.1415 upper=-3.1415 effort=1 velocity=1
- added joint 44_to_0: type revolute, parent 0, child 44, origin xyz=0.8496395744908001 0.7047834527789605 0.7132043539178358 rpy=16.614113858757964 5.9545604583241145 2.686502467429438, axis 1 0 0, limit lower=3.1415 upper=-3.1415 effort=1 velocity=1
- joint 11_to_0: axis 1 0 0 -> 0 0 1; origin xyz=0.7582277887228892 0.8648333499555793 0.721060376806119 rpy=7.249462115918347 0.133259755266637 5.237415269579376 -> xyz=0.9999 0.9999 0.3069430828837445 rpy=6.3641121477170985 6.282556988648868 6.282556988648868

File: L6/cm3020_ai/simscreatures/test.urdf (robot description, URDF)
Before this commit: robot pepe, 4 links, 3 joints
Links:
- removed link 12
- removed link 13
- added link 22, mass 2.341052065961812; collision cylinder length=0.7453290750283473 radius=0.9999; visual cylinder length=0.7453290750283473 radius=0.9999
- added link 33, mass 0.5256194207572338; collision cylinder length=0.8538696292666539 radius=0.4426546002600883; visual cylinder length=0.8538696292666539 radius=0.4426546002600883
- link 0: mass 0.2103234233305153 -> 3.1406502700383543; geometry collision cylinder length=0.9999 radius=0.9999; visual cylinder length=0.9999 radius=0.9999
- link 11: mass 2.297918675244149 -> 2.2929155202971745; geometry collision cylinder length=0.7300036717291499 radius=0.9999; visual cylinder length=0.7300036717291499 radius=0.9999
Joints:
- removed joint 12_to_0
- removed joint 13_to_0
- added joint 22_to_0: type revolute, parent 0, child 22, origin xyz=0.1311087775363201 0.3477177261943495 0.2820789912410324 rpy=5.448533740460787 1.2991002800413411 0.4333813206080416, axis 0 1 0, limit lower=3.1415 upper=-3.1415 effort=1 velocity=1
- added joint 33_to_0: type revolute, parent 0, child 33, origin xyz=0.6116192775281772 0.2640215550702885 0.8650797109700512 rpy=17.081542922329827 6.282556988648868 3.470044771954775, axis 0 1 0, limit lower=3.1415 upper=-3.1415 effort=1 velocity=1
- joint 11_to_0: axis 1 0 0 -> 0 0 1; origin xyz=0.8166271055768323 0.060541167397329065 0.9999 rpy=7.526699464513911 4.831392402738542 2.270539807682347 -> xyz=0.5001601937773651 0.9999 0.3908777749981114 rpy=12.565113977297736 3.4322828162417234 3.5980699676393
